File: _eagle/googleShoes.brd (EAGLE design)
At the start: 34.3 x 81.3 mm, 27 parts, among them U1 MCP73831, U2 3.3V, U3 ATMEGA328, Y1 8MHz

Commit message: added audio module
Parts:
- removed S1: (no value), SparkFun:TACTILE_SWITCH_SMD
- removed U$4: FIDUCIAL1X2, SparkFun:FIDUCIAL-1X2
- added D10, D2, D3, D5, D6, D7, D8, D9: LED, adafruit:CHIP-LED0805
- added JP7: FSR_BATT_CONNECT, SparkFun-Connectors:1X04
- added R2: 1Mohm, rcl:M0805
- added RN1, RN2: CTS742C083, resistor-net:CTS742C083
- C10, C2, C3, C6, C9: device SparkFun:0402-CAP -> adafruit:C0805
- D1: device led:LED5MM -> adafruit:CHIP-LED0805
- D4: device SparkFun:LED-0603 -> adafruit:CHIP-LED0805
- JP2: device SparkFun:1X02 -> SparkFun-Connectors:1X07
- JP3: device SparkFun:JST-2-SMD -> SparkFun-Connectors:1X07
- R1, R4, R5, R9: device SparkFun:0402-RES -> rcl:M0805
- moved JP3 25.2 mm to (19.1, 41.9)
- moved JP2 24.6 mm to (35.9, 41.9), flipped to the top
- moved D1 24.0 mm to (32.0, 57.3), turned to 90 degrees
- moved C1 19.8 mm to (35.9, 59.9), turned to 270 degrees
- moved JP5 19.0 mm to (8.13, 23.9)
- moved U3 18.3 mm to (24.6, 58.2)
- moved R5 17.7 mm to (13.8, 79.0), turned to 270 degrees
- moved JP4 17.2 mm to (35.8, 53.1), turned to 180 degrees
- moved U1 16.1 mm to (17.0, 78.9), turned to 0 degrees
- moved U2 14.9 mm to (35.8, 68.6)
- moved R1 14.7 mm to (32.0, 59.7), turned to 0 degrees
- moved R9 14.5 mm to (17.0, 75.3), turned to 0 degrees
- moved C2 14.3 mm to (31.9, 62.1)
- moved F1 13.9 mm to (27.8, 79.0), turned to 0 degrees
- moved D4 13.3 mm to (20.1, 79.0)
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Connections:
- new net N$13: D10.A, RN1.8
- new net N$15: D9.A, RN1.7
- new net N$16: D8.A, RN1.6
- new net N$17: D7.A, RN1.5
- new net N$3: D3.A, RN2.5
- new net N$4: D2.A, RN2.6
- new net N$6: D5.A, RN2.7
- new net N$7: D6.A, RN2.8
- new net SPK+: JP3.4
- new net SPK-: JP3.5
- net A0: now also JP7.4, R2.2
- net D2: now also JP3.3
- net D3: now also JP2.3
- net D4: now also JP2.4
- net D5: now also JP2.5
- net GND: now also D1.C, D10.C, D2.C, D3.C, D5.C, D6.C, D7.C, D8.C, D9.C, JP3.2, JP7.1, R2.1; no longer D1.K, JP2.1, JP3.1, S1.1, S1.2
- net RST: no longer S1.3, S1.4
- net VBATT: now also JP7.2; no longer JP2.2, JP3.2
- net VCC: now also JP3.1, JP7.3
Routing:
- net VCC: track 85.4 -> 0.00 mm, vias 6 -> 0
- net AREF: track 51.2 -> 0.00 mm, vias 3 -> 0
- net SCK: track 40.3 -> 0.00 mm, vias 4 -> 0
- net RXI: track 39.6 -> 0.00 mm, vias 2 -> 0
- net TXO: track 39.4 -> 0.00 mm, vias 2 -> 0
- net USB_VIN: track 36.8 -> 0.00 mm, vias 2 -> 0
- net RST: track 35.7 -> 0.00 mm
- net VBATT: track 25.1 -> 0.00 mm, vias 3 -> 0
- net N$5: track 21.1 -> 0.00 mm
- net MISO: track 19.0 -> 0.00 mm, vias 2 -> 0
- net N$12: track 14.5 -> 0.00 mm, vias 2 -> 0
- net N$2: track 13.4 -> 0.00 mm, vias 2 -> 0
- net A4: track 12.7 -> 0.00 mm, vias 2 -> 0
- net N$10: track 12.7 -> 0.00 mm
- net A5: track 11.7 -> 0.00 mm, vias 2 -> 0
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Other:
- board size 34.3 x 81.3 mm -> 38.1 x 81.3 mm

Commit message: added amplifier. needs routing.
Parts:
- added C4, C5, C7: 1uF, SparkFun:1206
- added C8: 10uF, SparkFun:1206
- added JP11: VOLUME, SparkFun:1X03
- added JP8: IN, SparkFun:1X02
- added JP9: OUT, SparkFun:1X02
- added LED1: (no value), led:CHIPLED_0805
- added Q1: MMBT2222A, SparkFun:SOT23-3
- added R10, R8: 150K, resistor:M0805
- added R3, R6: 10K, resistor:M0805
- added R7: 330, resistor:M0805
- added SJ1: (no value), SparkFun:SJ_2S-NOTRACE
- added U4: TPA2005D1DRB, mike-temp:QFN-8_PAD
- moved JP2 8.64 mm to (36.3, 33.3)
- moved JP3 8.64 mm to (19.4, 33.3)
- moved R2 5.09 mm to (23.6, 65.5), turned to 180 degrees
- moved D1 4.58 mm to (32.3, 61.8)
- moved R4 3.94 mm to (35.7, 64.6)
- moved C2 2.54 mm to (31.9, 64.6)
- moved C3 2.45 mm to (19.6, 65.4)
- moved JP4 2.22 mm to (36.3, 55.2)
- moved Y1 1.89 mm to (27.4, 51.8)
- moved R1 0.28 mm to (32.3, 59.8)
Connections:
- removed net SPK+: JP3.4
- removed net SPK-: JP3.5
- new net IN+: JP11.1, JP3.4, JP8.1, SJ1.2
- new net IN+AMP: R8.2, U4.3
- new net IN-: C7.1, JP11.3, JP3.5, JP8.2
- new net IN-AMP: R10.2, U4.4
- new net N$1: C5.1, JP11.2, SJ1.1
- new net N$18: LED1.A, R7.1
- new net N$19: Q1.1, R6.2
- new net N$20: LED1.C, Q1.3
- new net N$21: C5.2, R8.1
- new net N$22: C7.2, R10.1
- new net OUT+: JP9.1, U4.5
- new net OUT-: JP9.2, U4.8
- new net SDN*: R3.1, R6.1, U4.1
- net GND: now also C4.2, C8.2, Q1.2, U4.10, U4.11, U4.12, U4.13, U4.7
- net VCC: now also C4.1, C8.1, R3.2, R7.2, U4.6

Commit message: board layout
Parts:
- moved SJ1 7.87 mm to (19.9, 48.5)
- moved R8 5.68 mm to (27.9, 45.7)
- moved C5 5.08 mm to (24.9, 48.8)
- moved C8 3.75 mm to (23.2, 45.5)
- moved C4 3.59 mm to (23.2, 43.2)
- moved R7 1.25 mm to (36.3, 43.6), turned to 270 degrees
- moved Q1 1.17 mm to (30.4, 48.8), turned to 90 degrees
- moved U4 0.38 mm to (28.3, 42.7)
Changed lines of the file:
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@@
 <param name="mdSmdStop" value="0mil"/>
 <param name="msWidth" value="8mil"/>
-<param name="msDrill" value="20mil"/>
-<param name="msMicroVia" value="9.99mm"/>
+<param name="msDrill" value="8mil"/>
+<param name="msMicroVia" value="8mm"/>
 <param name="msBlindViaRatio" value="0.5"/>
 <param name="rvPadTop" value="0.25"/>
@@
 <element name="JP8" library="SparkFun" package="1X02" value="IN" x="19.05" y="41.91" rot="R90"/>
 <element name="JP9" library="SparkFun" package="1X02" value="OUT" x="1.27" y="2.54" rot="R90"/>
-<element name="C4" library="SparkFun" package="1206" value="1uF" x="25.146" y="46.228" rot="R180"/>
-<element name="C5" library="SparkFun" package="1206" value="1uF" x="19.812" y="48.768"/>
+<element name="C4" library="SparkFun" package="1206" value="1uF" x="23.241" y="43.18" rot="R180"/>
+<element name="C5" library="SparkFun" package="1206" value="1uF" x="24.892" y="48.768"/>
 <element name="C7" library="SparkFun" package="1206" value="1uF" x="35.306" y="47.117"/>
 <element name="R3" library="resistor" package="M0805" value="10K" x="33.02" y="42.545"/>
-<element name="Q1" library="SparkFun" package="SOT23-3" value="MMBT2222A" x="29.591" y="47.879"/>
+<element name="Q1" library="SparkFun" package="SOT23-3" value="MMBT2222A" x="30.353" y="48.768" rot="R90"/>
 <element name="R6" library="resistor" package="M0805" value="10K" x="33.02" y="40.64"/>
-<element name="R7" library="resistor" package="M0805" value="330" x="35.814" y="42.418" rot="R180"/>
+<element name="R7" library="resistor" package="M0805" value="330" x="36.322" y="43.561" rot="R270"/>
 <element name="LED1" library="led" package="CHIPLED_0805" value="" x="32.893" y="44.577" rot="R90"/>
-<element name="SJ1" library="SparkFun" package="SJ_2S-NOTRACE" value="" x="22.352" y="41.021" rot="R180"/>
+<element name="SJ1" library="SparkFun" package="SJ_2S-NOTRACE" value="" x="19.939" y="48.514" rot="R180"/>
 <element name="JP11" library="SparkFun" package="1X03" value="VOLUME" x="18.415" y="51.689"/>
-<element name="C8" library="SparkFun" package="1206" value="10uF" x="25.019" y="48.768" rot="R180"/>
-<element name="U4" library="mike-temp" package="QFN-8_PAD" value="TPA2005D1DRB" x="27.94" y="42.672" rot="R90"/>
-<element name="R8" library="resistor" package="M0805" value="150K" x="22.86" y="43.18"/>
+<element name="C8" library="SparkFun" package="1206" value="10uF" x="23.241" y="45.466" rot="R180"/>
+<element name="U4" library="mike-temp" package="QFN-8_PAD" value="TPA2005D1DRB" x="28.321" y="42.672" rot="R90"/>
+<element name="R8" library="resistor" package="M0805" value="150K" x="27.94" y="45.72"/>
 <element name="R10" library="resistor" package="M0805" value="150K" x="34.544" y="49.53" rot="R180"/>
 </elements>
@@
 <contactref element="C8" pad="2"/>
 <wire x1="4.665" y1="72.39" x2="6.32" y2="75.94" width="0" layer="19" extent="1-1"/>
+<wire x1="26.846" y1="42.347" x2="27.996" y2="41.2845" width="0" layer="19" extent="1-1"/>
 </signal>
 <signal name="VCC" class="1">
@@
 <wire x1="25.828" y1="53.8834" x2="26.628" y2="62.4686" width="0" layer="19" extent="1-1"/>
 <wire x1="24.228" y1="53.8834" x2="25.828" y2="53.8834" width="0" layer="19" extent="1-1"/>
-<wire x1="26.419" y1="48.768" x2="25.828" y2="53.8834" width="0" layer="19" extent="1-1"/>
-<wire x1="26.546" y1="46.228" x2="26.419" y2="48.768" width="0" layer="19" extent="1-1"/>
-<wire x1="26.465" y1="42.997" x2="26.546" y2="46.228" width="0" layer="19" extent="1-1"/>
-<wire x1="33.97" y1="42.545" x2="26.465" y2="42.997" width="0" layer="19" extent="1-1"/>
-<wire x1="34.864" y1="42.418" x2="33.97" y2="42.545" width="0" layer="19" extent="1-1"/>
-<wire x1="19.431" y1="33.274" x2="26.465" y2="42.997" width="0" layer="19" extent="1-1"/>
+<wire x1="24.641" y1="45.466" x2="24.228" y2="53.8834" width="0" layer="19" extent="1-1"/>
+<wire x1="24.641" y1="43.18" x2="24.641" y2="45.466" width="0" layer="19" extent="1-1"/>
+<wire x1="26.846" y1="42.997" x2="24.641" y2="43.18" width="0" layer="19" extent="1-1"/>
+<wire x1="33.97" y1="42.545" x2="26.846" y2="42.997" width="0" layer="19" extent="1-1"/>
+<wire x1="36.322" y1="42.611" x2="33.97" y2="42.545" width="0" layer="19" extent="1-1"/>
+<wire x1="19.431" y1="33.274" x2="24.641" y2="43.18" width="0" layer="19" extent="1-1"/>
 <wire x1="1.778" y1="23.876" x2="19.431" y2="33.274" width="0" layer="19" extent="1-1"/>
 <wire x1="10.414" y1="7.493" x2="1.778" y2="23.876" width="0" layer="19" extent="1-1"/>
@@
 <contactref element="JP9" pad="1"/>
 <contactref element="U4" pad="5"/>
-<wire x1="1.27" y1="2.54" x2="26.465" y2="43.647" width="0" layer="19" extent="1-1"/>
+<wire x1="1.27" y1="2.54" x2="26.846" y2="43.647" width="0" layer="19" extent="1-1"/>
 </signal>
 <signal name="OUT-">
 <contactref element="JP9" pad="2"/>
 <contactref element="U4" pad="8"/>
-<wire x1="1.27" y1="5.08" x2="26.465" y2="41.697" width="0" layer="19" extent="1-1"/>
+<wire x1="1.27" y1="5.08" x2="26.846" y2="41.697" width="0" layer="19" extent="1-1"/>
 </signal>
 <signal name="SDN*">
@@
 <contactref element="R6" pad="1"/>
 <wire x1="32.07" y1="40.64" x2="32.07" y2="42.545" width="0" layer="19" extent="1-1"/>
-<wire x1="29.415" y1="41.697" x2="32.07" y2="42.545" width="0" layer="19" extent="1-1"/>
+<wire x1="29.796" y1="41.697" x2="32.07" y2="42.545" width="0" layer="19" extent="1-1"/>
 </signal>
 <signal name="N$1">
@@
 <contactref element="SJ1" pad="1"/>
 <contactref element="JP11" pad="2"/>
-<wire x1="18.412" y1="48.768" x2="20.955" y2="51.689" width="0" layer="19" extent="1-1"/>
-<wire x1="22.7529" y1="41.021" x2="18.412" y2="48.768" width="0" layer="19" extent="1-1"/>
+<wire x1="20.3399" y1="48.514" x2="23.492" y2="48.768" width="0" layer="19" extent="1-1"/>
+<wire x1="20.955" y1="51.689" x2="20.3399" y2="48.514" width="0" layer="19" extent="1-1"/>
 </signal>
 <signal name="IN-AMP">
 <contactref element="R10" pad="2"/>
 <contactref element="U4" pad="4"/>
-<wire x1="29.415" y1="43.647" x2="33.594" y2="49.53" width="0" layer="19" extent="1-1"/>
+<wire x1="29.796" y1="43.647" x2="33.594" y2="49.53" width="0" layer="19" extent="1-1"/>
 </signal>
 <signal name="N$18">
 <contactref element="R7" pad="1"/>
 <contactref element="LED1" pad="A"/>
-<wire x1="33.943" y1="44.577" x2="36.764" y2="42.418" width="0" layer="19" extent="1-1"/>
+<wire x1="33.943" y1="44.577" x2="36.322" y2="44.511" width="0" layer="19" extent="1-1"/>
 </signal>
 <signal name="N$19">
 <contactref element="R6" pad="2"/>
 <contactref element="Q1" pad="1"/>
-<wire x1="28.641" y1="46.879" x2="33.97" y2="40.64" width="0" layer="19" extent="1-1"/>
+<wire x1="33.97" y1="40.64" x2="31.353" y2="47.818" width="0" layer="19" extent="1-1"/>
 </signal>
 <signal name="N$20">
 <contactref element="Q1" pad="3"/>
 <contactref element="LED1" pad="C"/>
-<wire x1="31.843" y1="44.577" x2="29.591" y2="48.979" width="0" layer="19" extent="1-1"/>
+<wire x1="31.843" y1="44.577" x2="29.253" y2="48.768" width="0" layer="19" extent="1-1"/>
 </signal>
 <signal name="IN+AMP">
 <contactref element="U4" pad="3"/>
 <contactref element="R8" pad="2"/>
-<wire x1="23.81" y1="43.18" x2="29.415" y2="42.997" width="0" layer="19" extent="1-1"/>
+<wire x1="29.796" y1="42.997" x2="28.89" y2="45.72" width="0" layer="19" extent="1-1"/>
 </signal>
 <signal name="N$21">
 <contactref element="R8" pad="1"/>
 <contactref element="C5" pad="2"/>
-<wire x1="21.91" y1="43.18" x2="21.212" y2="48.768" width="0" layer="19" extent="1-1"/>
+<wire x1="26.99" y1="45.72" x2="26.292" y2="48.768" width="0" layer="19" extent="1-1"/>
 </signal>
 <signal name="N$22">
@@
 <contactref element="SJ1" pad="2"/>
 <contactref element="JP11" pad="1"/>
-<wire x1="19.05" y1="41.91" x2="18.415" y2="51.689" width="0" layer="19" extent="1-1"/>
-<wire x1="21.9393" y1="41.021" x2="19.05" y2="41.91" width="0" layer="19" extent="1-1"/>
-<wire x1="19.431" y1="25.654" x2="21.9393" y2="41.021" width="0" layer="19" extent="1-1"/>
+<wire x1="19.5263" y1="48.514" x2="18.415" y2="51.689" width="0" layer="19" extent="1-1"/>
+<wire x1="19.05" y1="41.91" x2="19.5263" y2="48.514" width="0" layer="19" extent="1-1"/>
+<wire x1="19.431" y1="25.654" x2="19.05" y2="41.91" width="0" layer="19" extent="1-1"/>
 </signal>
 </signals>

Commit message: routed again- rev02
Parts:
- moved C5 2.92 mm to (23.2, 46.4)
- moved C8 1.27 mm to (23.2, 44.2)
- moved C4 1.14 mm to (23.2, 42.0)
- moved LED1 0.63 mm to (33.5, 44.6)
- moved R3 0.52 mm to (33.5, 42.7)
- moved R6 0.51 mm to (33.5, 40.6)
- moved R7 0.38 mm to (36.7, 43.6)
- moved R8 0.36 mm to (28.2, 46.0)
Changed lines of the file:
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@@
 <element name="JP8" library="SparkFun" package="1X02" value="IN" x="19.05" y="41.91" rot="R90"/>
 <element name="JP9" library="SparkFun" package="1X02" value="OUT" x="1.27" y="2.54" rot="R90"/>
-<element name="C4" library="SparkFun" package="1206" value="1uF" x="23.241" y="43.18" rot="R180"/>
-<element name="C5" library="SparkFun" package="1206" value="1uF" x="24.892" y="48.768"/>
+<element name="C4" library="SparkFun" package="1206" value="1uF" x="23.241" y="42.037" rot="R180"/>
+<element name="C5" library="SparkFun" package="1206" value="1uF" x="23.241" y="46.355"/>
 <element name="C7" library="SparkFun" package="1206" value="1uF" x="35.306" y="47.117"/>
-<element name="R3" library="resistor" package="M0805" value="10K" x="33.02" y="42.545"/>
+<element name="R3" library="resistor" package="M0805" value="10K" x="33.528" y="42.672"/>
 <element name="Q1" library="SparkFun" package="SOT23-3" value="MMBT2222A" x="30.353" y="48.768" rot="R90"/>
-<element name="R6" library="resistor" package="M0805" value="10K" x="33.02" y="40.64"/>
-<element name="R7" library="resistor" package="M0805" value="330" x="36.322" y="43.561" rot="R270"/>
-<element name="LED1" library="led" package="CHIPLED_0805" value="" x="32.893" y="44.577" rot="R90"/>
+<element name="R6" library="resistor" package="M0805" value="10K" x="33.528" y="40.64"/>
+<element name="R7" library="resistor" package="M0805" value="330" x="36.703" y="43.561" rot="R270"/>
+<element name="LED1" library="led" package="CHIPLED_0805" value="" x="33.528" y="44.577" rot="R90"/>
 <element name="SJ1" library="SparkFun" package="SJ_2S-NOTRACE" value="" x="19.939" y="48.514" rot="R180"/>
 <element name="JP11" library="SparkFun" package="1X03" value="VOLUME" x="18.415" y="51.689"/>
-<element name="C8" library="SparkFun" package="1206" value="10uF" x="23.241" y="45.466" rot="R180"/>
+<element name="C8" library="SparkFun" package="1206" value="10uF" x="23.241" y="44.196" rot="R180"/>
 <element name="U4" library="mike-temp" package="QFN-8_PAD" value="TPA2005D1DRB" x="28.321" y="42.672" rot="R90"/>
-<element name="R8" library="resistor" package="M0805" value="150K" x="27.94" y="45.72"/>
+<element name="R8" library="resistor" package="M0805" value="150K" x="28.194" y="45.974"/>
 <element name="R10" library="resistor" package="M0805" value="150K" x="34.544" y="49.53" rot="R180"/>
 </elements>
@@
 <wire x1="25.828" y1="53.8834" x2="26.628" y2="62.4686" width="0" layer="19" extent="1-1"/>
 <wire x1="24.228" y1="53.8834" x2="25.828" y2="53.8834" width="0" layer="19" extent="1-1"/>
-<wire x1="24.641" y1="45.466" x2="24.228" y2="53.8834" width="0" layer="19" extent="1-1"/>
-<wire x1="24.641" y1="43.18" x2="24.641" y2="45.466" width="0" layer="19" extent="1-1"/>
-<wire x1="26.846" y1="42.997" x2="24.641" y2="43.18" width="0" layer="19" extent="1-1"/>
-<wire x1="33.97" y1="42.545" x2="26.846" y2="42.997" width="0" layer="19" extent="1-1"/>
-<wire x1="36.322" y1="42.611" x2="33.97" y2="42.545" width="0" layer="19" extent="1-1"/>
-<wire x1="19.431" y1="33.274" x2="24.641" y2="43.18" width="0" layer="19" extent="1-1"/>
+<wire x1="24.641" y1="44.196" x2="24.228" y2="53.8834" width="0" layer="19" extent="1-1"/>
+<wire x1="24.641" y1="42.037" x2="24.641" y2="44.196" width="0" layer="19" extent="1-1"/>
+<wire x1="26.846" y1="42.997" x2="24.641" y2="42.037" width="0" layer="19" extent="1-1"/>
+<wire x1="34.478" y1="42.672" x2="26.846" y2="42.997" width="0" layer="19" extent="1-1"/>
+<wire x1="36.703" y1="42.611" x2="34.478" y2="42.672" width="0" layer="19" extent="1-1"/>
+<wire x1="19.431" y1="33.274" x2="24.641" y2="42.037" width="0" layer="19" extent="1-1"/>
 <wire x1="1.778" y1="23.876" x2="19.431" y2="33.274" width="0" layer="19" extent="1-1"/>
 <wire x1="10.414" y1="7.493" x2="1.778" y2="23.876" width="0" layer="19" extent="1-1"/>
@@
 <contactref element="U4" pad="1"/>
 <contactref element="R6" pad="1"/>
-<wire x1="32.07" y1="40.64" x2="32.07" y2="42.545" width="0" layer="19" extent="1-1"/>
-<wire x1="29.796" y1="41.697" x2="32.07" y2="42.545" width="0" layer="19" extent="1-1"/>
+<wire x1="32.578" y1="40.64" x2="32.578" y2="42.672" width="0" layer="19" extent="1-1"/>
+<wire x1="29.796" y1="41.697" x2="32.578" y2="42.672" width="0" layer="19" extent="1-1"/>
 </signal>
 <signal name="N$1">
@@
 <contactref element="SJ1" pad="1"/>
 <contactref element="JP11" pad="2"/>
-<wire x1="20.3399" y1="48.514" x2="23.492" y2="48.768" width="0" layer="19" extent="1-1"/>
+<wire x1="20.3399" y1="48.514" x2="21.841" y2="46.355" width="0" layer="19" extent="1-1"/>
 <wire x1="20.955" y1="51.689" x2="20.3399" y2="48.514" width="0" layer="19" extent="1-1"/>
 </signal>
@@
 <contactref element="R7" pad="1"/>
 <contactref element="LED1" pad="A"/>
-<wire x1="33.943" y1="44.577" x2="36.322" y2="44.511" width="0" layer="19" extent="1-1"/>
+<wire x1="34.578" y1="44.577" x2="36.703" y2="44.511" width="0" layer="19" extent="1-1"/>
 </signal>
 <signal name="N$19">
 <contactref element="R6" pad="2"/>
 <contactref element="Q1" pad="1"/>
-<wire x1="33.97" y1="40.64" x2="31.353" y2="47.818" width="0" layer="19" extent="1-1"/>
+<wire x1="34.478" y1="40.64" x2="31.353" y2="47.818" width="0" layer="19" extent="1-1"/>
 </signal>
 <signal name="N$20">
 <contactref element="Q1" pad="3"/>
 <contactref element="LED1" pad="C"/>
-<wire x1="31.843" y1="44.577" x2="29.253" y2="48.768" width="0" layer="19" extent="1-1"/>
+<wire x1="32.478" y1="44.577" x2="29.253" y2="48.768" width="0" layer="19" extent="1-1"/>
 </signal>
 <signal name="IN+AMP">
 <contactref element="U4" pad="3"/>
 <contactref element="R8" pad="2"/>
-<wire x1="29.796" y1="42.997" x2="28.89" y2="45.72" width="0" layer="19" extent="1-1"/>
+<wire x1="29.796" y1="42.997" x2="29.144" y2="45.974" width="0" layer="19" extent="1-1"/>
 </signal>
 <signal name="N$21">
 <contactref element="R8" pad="1"/>
 <contactref element="C5" pad="2"/>
-<wire x1="26.99" y1="45.72" x2="26.292" y2="48.768" width="0" layer="19" extent="1-1"/>
+<wire x1="27.244" y1="45.974" x2="24.641" y2="46.355" width="0" layer="19" extent="1-1"/>
 </signal>
 <signal name="N$22">
