File: _eagle/googleShoes_rev02.brd (EAGLE design)
At the start: 38.1 x 81.3 mm, 53 parts, among them Q1 MMBT2222A, U1 MCP73831, U2 3.3V, U3 ATMEGA328, U4 TPA2005D1DRB, Y1 8MHz

Commit message: routed again- rev02
Parts:
- moved SJ1 7.87 mm to (19.9, 48.5)
- moved R8 6.02 mm to (28.2, 46.0)
- moved C5 3.69 mm to (23.5, 48.6)
- moved C4 3.10 mm to (23.4, 43.7)
- moved C8 3.00 mm to (23.2, 46.4)
- moved R7 1.45 mm to (36.7, 43.6), turned to 270 degrees
- moved Q1 1.17 mm to (30.4, 48.8), turned to 90 degrees
- moved LED1 0.63 mm to (33.5, 44.6)
- moved R3 0.52 mm to (33.5, 42.7)
- moved R6 0.51 mm to (33.5, 40.6)
- moved U4 0.38 mm to (28.3, 42.7)
Routing:
- net VCC: track 0.00 -> 195.8 mm, vias 0 -> 8
- net VBATT: track 0.00 -> 96.2 mm, vias 0 -> 9
- net OUT+: track 0.00 -> 70.6 mm, vias 0 -> 4
- net A0: track 0.00 -> 69.7 mm, vias 0 -> 6
- net OUT-: track 0.00 -> 60.3 mm, vias 0 -> 4
- net D4: track 0.00 -> 58.0 mm, vias 0 -> 4
- net IN-: track 0.00 -> 51.4 mm, vias 0 -> 3
- net D3: track 0.00 -> 47.0 mm, vias 0 -> 2
- net A5: track 0.00 -> 44.3 mm, vias 0 -> 2
- net A4: track 0.00 -> 43.1 mm, vias 0 -> 2
- net D5: track 0.00 -> 39.9 mm, vias 0 -> 2
- net RST: track 0.00 -> 33.6 mm, vias 0 -> 2
- net D2: track 0.00 -> 32.3 mm, vias 0 -> 2
- net AREF: track 0.00 -> 30.9 mm, vias 0 -> 2
- net USB_VIN: track 0.00 -> 30.1 mm, vias 0 -> 4
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